File: hardware/amplifier2/amplifier.kicad_pcb (KiCad board)
At the start: 2 copper layers, 95 x 82 mm, 132 parts, among them IC1 AD8331, IC2 ISL55210, IC3 LP38798, IC4 NC7SVU04, IC5 LTC2252, J1 0, M1 MountingHole_3.2mm_M3_Pad, M2 MountingHole_3.2mm_M3_Pad, M3 MountingHole_3.2mm_M3_Pad, M4 MountingHole_3.2mm_M3_Pad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

Commit message: minor fixes mr. hufschmid mentioned
Parts:
- T1, T2, T3, T4: footprint SDRfootprints:CX2041NLT -> SDRfootprints:T4-1-KK81
- moved C21 8.51 mm to (170.6, 74.9)
- moved C22 8.51 mm to (168.6, 84.5)
- moved C23 8.51 mm to (168.3, 78.6)
- moved C24 8.51 mm to (175.8, 83.0)
- moved C25 8.51 mm to (173.7, 79.0)
- moved IC2 8.51 mm to (168.1, 80.7)
- moved L5 8.51 mm to (168.6, 86.1)
- moved L6 8.51 mm to (168.3, 77.0)
- moved R10 8.51 mm to (166.0, 80.1)
- moved R11 8.51 mm to (166.0, 82.7)
- moved R12 8.51 mm to (170.6, 77.7)
- moved R13 8.51 mm to (173.7, 82.2)
- moved R14 8.51 mm to (173.7, 80.6)
- moved R9 8.51 mm to (170.9, 85.6)
- moved R36 6.71 mm to (174.6, 97.6)
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Connections:
- R17 pad 1: /OUT2- -> /OUT2+
- R18 pad 1: /OUT2+ -> /OUT2-
- R37 pad 1: /IN2+ -> /IN2-
- R38 pad 1: /IN2- -> /IN2+
- R5 pad 1: /OUT1- -> /OUT1+
- R6 pad 1: /OUT1+ -> /OUT1-
Routing:
- net GNDA: track 368.9 -> 323.9 mm, vias 301 -> 260
- net Net-(T4-Pad1): track 9.02 -> 24.7 mm
- net Net-(R6-Pad2): track 2.05 -> 14.6 mm
- net Net-(R37-Pad2): track 2.32 -> 13.0 mm
- net Net-(T1-Pad1): track 8.51 -> 17.4 mm
- net Net-(R17-Pad2): track 2.69 -> 11.6 mm
- net Net-(R5-Pad2): track 2.07 -> 10.8 mm
- net /IN2+: track 45.8 -> 54.4 mm
- net /IN2-: track 51.9 -> 59.9 mm
- net Net-(T2-Pad1): track 9.95 -> 17.2 mm
- net (no net): track 0.00 -> 6.88 mm, vias 0 -> 6
- net Net-(C30-Pad1): track 12.4 -> 17.7 mm
- net /OUT2-: track 18.4 -> 14.2 mm
- net Net-(R38-Pad2): track 2.26 -> 6.33 mm
- net Net-(R18-Pad2): track 2.30 -> 6.37 mm
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