File: hardware/amplifier2/amplifier.sch (KiCad schematic (older format))
At the start: 128 parts, among them IC1 AD8331, IC2 ISL55210, IC3 LP38798, IC4 NC7SVU04, IC5 LTC2252, J1 0, P1 5V, P2 UART, P4 VGA - LNA, P5 LNA - SDR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

Commit message: beautified and corrected bom; added aufgabenstellung; added both to report
Parts:
- L3, L4: footprint SDRfootprints:COIL_445-4177-1-ND -> Choke_SMD:Choke_SMD_1206_Standard
Changed lines of the file:
@@
 F 0 "L3" V 4935 1150 50  0000 C CNN
 F 1 "22u" V 4844 1150 50  0000 C CNN
-F 2 "SDRfootprints:COIL_445-4177-1-ND" H 4750 1150 50  0001 C CNN
+F 2 "Choke_SMD:Choke_SMD_1206_Standard" H 4750 1150 50  0001 C CNN
 F 3 "" H 4750 1150 50  0000 C CNN
 	1    4750 1150
@@
 F 0 "L4" V 6235 1150 50  0000 C CNN
 F 1 "22u" V 6144 1150 50  0000 C CNN
-F 2 "SDRfootprints:COIL_445-4177-1-ND" H 6050 1150 50  0001 C CNN
+F 2 "Choke_SMD:Choke_SMD_1206_Standard" H 6050 1150 50  0001 C CNN
 F 3 "" H 6050 1150 50  0000 C CNN
 	1    6050 1150
