File: hardware/amplifier2-pcb1/amplifier.sch (KiCad schematic (older format))
At the start: 128 parts, among them IC1 AD8331, IC2 ISL55210, IC3 LP38798, IC4 NC7SVU04, IC5 LTC2252, J1 0, P1 5V, P2 UART, P4 VGA - LNA, P5 LNA - SDR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

Commit message: Duplicated amp schematics for version1 so version2 can be edited already; added jupyter nb for measuring and evaluation; added pdf for bom; added arduino software to speak to dac
Other:
- note removed: "Possibly needs to be fed from 5V net!"
Changed lines of the file:
@@
 Text Notes 16950 11100 0    197  ~ 0
 The ADC part has also been included.\nIt has a groundplane as close as possible to the one in the app. note.\nAdiddionally the pre-ADC circuitry can now thoroughly be tested.
-Wire Notes Line
-	3200 10450 3200 12400
-Wire Notes Line
-	3200 12400 800  12400
-Text Notes 800  12400 0    60   ~ 0
-Possibly needs to be fed from 5V net!
-Wire Notes Line
-	3200 10650 2350 10650
-Wire Notes Line
-	2350 10650 2350 10050
-Wire Notes Line
-	2150 10000 2150 10050
-Wire Notes Line
-	2150 10050 2550 10050
-Wire Notes Line
-	2550 10050 2550 10000
 $EndSCHEMATC
